File: sw-4416-project-v1.sch (EAGLE design)
At the start: 14 parts, among them IC1 MCP73833-UN, X1 USB-MICROB

Commit message: Added power circuitry
Parts:
- added C4, C5, C6, C7, C8, C9: 4.7uF, SparkFun:CAP0603-CAP
- added CN1: (no value), adafruit:JST_2PIN-SMT-RA
- added ISP1: AVRISP-6, adafruit:AVRISP-6
- added LED3: Green, SparkFun:LED0603
- added R4: 2k, SparkFun:RESISTOR0603-RES
- added R5: 330, SparkFun:RESISTOR0603-RES
- added R6: 390, SparkFun:RESISTOR0603-RES
- added R7: 240, SparkFun:RESISTOR0603-RES
- added R8, R9: 22, SparkFun:RESISTOR0603-RES
- added U1: V_REG_317SMD, SparkFun:V_REG_317SMD
- IC1: value MCP73833-UN -> MCP73831; device adafruit:MCP73833-UN -> SparkFun:MCP73831
Connections:
- new net 3.3V: C9.1, R7.2, U1.OUT
- new net N$10: R8.2, U$2.D-
- new net N$11: C5.1, CN1.2, IC1.VBAT, U1.IN
- new net N$12: R6.1, R7.1, U1.ADJ
- new net N$6: IC1.PROG, R4.2
- new net N$7: IC1.STAT, R5.2
- new net N$8: LED3.C, R5.1
- new net N$9: R9.2, U$2.D+
- new net VBUS: C4.1, IC1.VIN, LED3.A, X1.VBUS
- net GND: now also C4.2, C5.2, C6.2, C7.2, C8.2, C9.2, CN1.1, IC1.VSS, R4.1, R6.2; no longer IC1.GND
- net USB_D+: now also R9.1, X1.D+; no longer U$2.D+
- net USB_D-: now also R8.1, X1.D-; no longer U$2.D-
- net VCC: now also C6.1, C7.1, C8.1
