File: hardware/sw-4416-project-v1.brd (EAGLE design)
At the start: 100 x 80 mm, 58 parts, among them IC1 MCP73831, U1 ADP3338, X1 USB-MICROB, Y1 16M

Commit message: rev 1 board finished
Parts:
- removed JP8: JUMPER-3PTH, SparkFun:1X03
- removed U$4: LIPO-OUTLINE1100, SparkFun:LIPO-1100
- moved R14 154.5 mm to (76.2, 62.2), turned to 270 degrees
- moved C7 149.5 mm to (80.0, 63.5)
- moved R15 145.9 mm to (59.7, 45.7), turned to 180 degrees
- moved R13 135.8 mm to (59.7, 55.9), turned to 180 degrees
- moved C10 134.0 mm to (44.5, 30.5), turned to 180 degrees
- moved R2 126.4 mm to (86.4, 39.4)
- moved C8 126.3 mm to (52.1, 58.4), turned to 180 degrees
- moved R10 123.8 mm to (54.6, 43.2), turned to 90 degrees
- moved R1 119.9 mm to (82.5, 38.1), turned to 270 degrees
- moved U$2 118.2 mm to (41.9, 52.1)
- moved C6 117.0 mm to (52.1, 74.9), turned to 90 degrees
- moved R11 116.6 mm to (41.9, 40.6)
- moved R3 116.5 mm to (71.1, 38.1), turned to 270 degrees
- moved LED2 115.9 mm to (76.2, 38.1), turned to 180 degrees
- moved LED1 114.8 mm to (78.7, 38.1), turned to 180 degrees
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Connections:
- net XOUT: no longer JP8.3
- net YOUT: no longer JP8.2
- net ZOUT: no longer JP8.1
Routing:
- net GND: track 0.00 -> 437.8 mm, vias 0 -> 7
- net 3.3V: track 0.00 -> 201.9 mm, vias 0 -> 4
- net VUSB: track 0.00 -> 72.2 mm, vias 0 -> 2
- net N$17: track 0.00 -> 62.9 mm, vias 0 -> 3
- net VCC: track 0.00 -> 54.8 mm
- net ST: track 0.00 -> 53.3 mm, vias 0 -> 2
- net MCU_RST: track 0.00 -> 44.2 mm, vias 0 -> 1
- net BT_TX: track 0.00 -> 38.8 mm
- net BT_RST: track 0.00 -> 38.6 mm, vias 0 -> 2
- net XOUT: track 0.00 -> 32.7 mm
- net BT_RX: track 0.00 -> 32.6 mm
- net MOSI: track 0.00 -> 28.6 mm, vias 0 -> 1
- net YOUT: track 0.00 -> 27.5 mm
- net N$15: track 0.00 -> 25.8 mm, vias 0 -> 2
- net SCK: track 0.00 -> 23.6 mm
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- added copper zone on layer 16, net GND
- added copper zone on layer 1, net N$11
- added copper zone on layer 1, net N$29
- added copper zone on layer 1, net VCC
- added copper zone on layer 1, net VUSB
Other:
- board size 100 x 80 mm -> 94 x 52.1 mm
- board text added: "AREF"
- board text added: "DBG0"
- board text added: "DBG1"
- board text added: "Gnd"
- board text added: "Pwr"
- board text added: "RX"
- board text added: "TX"
- board text added: "UART"
- board text added: "USB"
- board text added: "USBPwr"
- board text added: "Vbat"

Commit message: working on embedded side code
Parts:
- added U$4: (no value), SparkFun:OSHW-LOGO-M
- moved CN1 1.27 mm to (26.7, 74.9)
Connections:
- net N$11 renamed VIN
Routing:
- net MCU_RST: track 44.2 -> 38.8 mm
- net 3.3V: track 201.9 -> 200.3 mm
- net ST: track 53.3 -> 54.0 mm
- net GND: track 437.8 -> 437.2 mm
- added copper zone on layer 1, net GND
- removed copper zone on layer 1, net N$29
- removed copper zone on layer 1, net VIN
Other:
- board size 94 x 52.1 mm -> 94 x 53.3 mm
- board text added: "3V3"
- board text added: "S. Watson"
- board text added: "sw-4416-project-v1"
