File: hardware/sw-4416-project-v1.sch (EAGLE design)
At the start: 30 parts, among them IC1 MCP73831, U1 V_REG_317SMD, X1 USB-MICROB

Commit message: schematic version 1 completed
Parts:
- added C10, C11: 22pF, SparkFun:CAP0603-CAP
- added C12, C13: 1uF, SparkFun:CAP0603-CAP
- added JP1: Vcc, SparkFun:JUMPER-2PTH
- added JP2: VUSB, SparkFun:JUMPER-2PTH
- added JP3: 3.3V, SparkFun:JUMPER-2PTH
- added JP4: GND, SparkFun:JUMPER-2PTH
- added JP5: AREF, SparkFun:JUMPER-2PTH
- added JP6: UART, SparkFun:JUMPER-2PTH
- added JP7: USB, SparkFun:JUMPER-2PTH
- added JP8: JUMPER-3PTH, SparkFun:JUMPER-3PTH
- added L1: (no value), SparkFun:INDUCTOR0805
- added LED4: Power, SparkFun:LED0603
- added LED5: RX, SparkFun:LED0603
- added LED6: TX, SparkFun:LED0603
- added LED7: DBG0, SparkFun:LED0603
- added LED8: DBG1, SparkFun:LED0603
- added R10, R15, R16: 330, SparkFun:RESISTOR0603-RES
- added R11: 1M, SparkFun:RESISTOR0603-RES
- added R12, R13, R14, R17: 10K, SparkFun:RESISTOR0603-RES
- added S1: Power, SparkFun:SWITCH-SPST-SMD-A
- added Y1: 16M, SparkFun:CRYSTALHC49US
- R6: value 390 -> 330
- R7: value 240 -> 330
- U1: value V_REG_317SMD -> ADP3338; device SparkFun:V_REG_317SMD -> dp_devices:VREG_3PINS-SOT-223
Connections:
- removed net VBUS: C4.1, IC1.VIN, LED3.A, X1.VBUS
- new net AREF: JP5.1, JP5.2, U$2.AREF
- new net DBG0: LED7.A, U$2.PB5(OC1A/ADC12/!OC4B)
- new net DBG1: LED8.A, U$2.PB6(OC1B/OC4B/ADC13)
- new net MCU_RST: ISP1.RST, R12.1, U$2./RESET
- new net MISO: ISP1.MISO, U$2.PB3(PDO/MISO)
- new net MOSI: ISP1.MOSI, U$2.PB2(PDI/MOSI)
- new net N$13: C10.1, R11.2, U$2.XTAL1, Y1.1
- new net N$14: C11.1, R11.1, U$2.XTAL2, Y1.2
- new net N$15: R8.2, X1.D+
- new net N$16: LED7.C, R15.2
- new net N$17: C13.2, L1.1, U$2.AVCC, U$2.AVCC1
- new net N$18: LED8.C, R16.2
- new net N$19: R13.2, U$2.PE2(!HWB)
- new net N$20: R9.2, X1.D-
- new net RX_LED: LED5.A, U$2.PB0(SS)
- new net SCK: ISP1.SCK, U$2.PB1(SCK)
- new net TX_LED: LED6.A, U$2.PD5(XCK/CTS)
- new net VUSB: C4.1, IC1.VIN, JP2.1, JP2.2, LED3.A, U$2.VBUS, X1.VBUS
- net 3.3V: now also C12.2, C6.1, C7.1, C8.2, ISP1.VCC, JP3.1, JP3.2, L1.2, LED4.A, R12.2, R14.1, U$1.VS@14, U$2.UCAP, U$2.VCC, U$2.VCC1, U$3.VDD, U1.VOUT; no longer R7.2, U1.OUT
- net BT_RST: now also R14.2, U$2.PB4(ADC11)
- net BT_RX: now also JP6.2
- net BT_TX: now also JP6.1
- net GND: now also C10.2, C11.2, C12.1, C13.1, C8.1, ISP1.GND, JP4.1, JP4.2, R10.1, R13.1, R15.1, R16.1, R17.2, R6.1, R7.1, U$2.UGND, U1.GND; no longer C8.2, R6.2
- net N$10: now also LED5.C, R7.2; no longer R8.2, U$2.D-
- net N$11: now also S1.O, U1.VIN; no longer C5.1, CN1.2, IC1.VBAT, U1.IN
- net N$12: now also LED6.C, R10.2; no longer R6.1, R7.1, U1.ADJ
- net N$9: now also LED4.C, R6.2; no longer R9.2, U$2.D+
- net ST: now also R17.1, U$2.PB7(OC0A/OC1C/RTS)
- net USB_D+: now also JP7.2, R8.1, U$2.D+; no longer R9.1, X1.D+
- net USB_D-: now also JP7.1, R9.1, U$2.D-; no longer R8.1, X1.D-
- net VCC: now also C5.1, CN1.2, IC1.VBAT, JP1.1, JP1.2, S1.P; no longer C6.1, C7.1, C8.1, U$1.VS@14, U$2.VCC, U$2.VCC1, U$3.VDD
- net XOUT: now also JP8.3
- net YOUT: now also JP8.2
- net ZOUT: now also JP8.1
Other:
- note added: "Battery & Charging"
- note added: "Debug"
- note added: "ICSP"
- note added: "Regulator"
- note added: "Sep 24/12"
- note added: "USB"
- note removed: "Power"
- moved on the sheet: C1, C2, C3, C4, C5, C6, C7, C8, C9, CN1, IC1, ISP1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

Commit message: rev 1 board finished
Parts:
- removed JP8: JUMPER-3PTH, SparkFun:JUMPER-3PTH
- removed U$4: LIPO-OUTLINE1100, SparkFun:LIPO-OUTLINE1100
Connections:
- net XOUT: no longer JP8.3
- net YOUT: no longer JP8.2
- net ZOUT: no longer JP8.1
Changed lines of the file:
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@@
 <setting verticaltext="up"/>
 </settings>
-<grid distance="0.1" unitdist="inch" unit="inch" style="lines" multiple="1" display="yes" altdistance="0.01" altunitdist="inch" altunit="inch"/>
+<grid distance="0.1" unitdist="inch" unit="inch" style="lines" multiple="1" display="no" altdistance="0.01" altunitdist="inch" altunit="inch"/>
 <layers>
 <layer number="1" name="Top" color="4" fill="1" visible="no" active="no"/>
@@
 <part name="U$2" library="adafruit" deviceset="ATMEGA32U4" device="-AU"/>
 <part name="U$3" library="SparkFun" deviceset="BLUETOOTH-RN41" device="&quot;"/>
-<part name="U$4" library="SparkFun" deviceset="LIPO-OUTLINE" device="1100"/>
 <part name="IC1" library="SparkFun" deviceset="MCP73831" device=""/>
 <part name="GND2" library="SparkFun" deviceset="GND" device=""/>
@@
 <part name="JP6" library="SparkFun" deviceset="JUMPER-2" device="PTH" value="UART"/>
 <part name="JP7" library="SparkFun" deviceset="JUMPER-2" device="PTH" value="USB"/>
-<part name="JP8" library="SparkFun" deviceset="JUMPER-3" device="PTH"/>
 <part name="P+2" library="SparkFun" deviceset="3.3V" device=""/>
 <part name="P+3" library="SparkFun" deviceset="3.3V" device=""/>
@@
 <instance part="U$2" gate="G$1" x="81.28" y="124.46"/>
 <instance part="U$3" gate="G$1" x="177.8" y="142.24"/>
-<instance part="U$4" gate="G$1" x="187.96" y="81.28" rot="R270"/>
 <instance part="IC1" gate="G$1" x="157.48" y="81.28"/>
 <instance part="GND2" gate="1" x="116.84" y="55.88"/>
@@
 <instance part="JP6" gate="A" x="91.44" y="25.4" rot="R90"/>
 <instance part="JP7" gate="A" x="91.44" y="12.7" rot="R90"/>
-<instance part="JP8" gate="G$1" x="119.38" y="12.7" rot="R90"/>
 <instance part="P+2" gate="G$1" x="12.7" y="73.66"/>
 <instance part="P+3" gate="G$1" x="48.26" y="157.48"/>
@@
 <label x="116.84" y="154.94" size="1.778" layer="95"/>
 </segment>
-<segment>
-<pinref part="JP8" gate="G$1" pin="3"/>
-<wire x1="121.92" y1="17.78" x2="127" y2="17.78" width="0.1524" layer="91"/>
-<label x="127" y="17.78" size="1.778" layer="95"/>
-</segment>
 </net>
 <net name="YOUT" class="0">
@@
 <label x="116.84" y="157.48" size="1.778" layer="95"/>
 </segment>
-<segment>
-<pinref part="JP8" gate="G$1" pin="2"/>
-<wire x1="121.92" y1="15.24" x2="127" y2="15.24" width="0.1524" layer="91"/>
-<label x="127" y="15.24" size="1.778" layer="95"/>
-</segment>
 </net>
 <net name="ZOUT" class="0">
@@
 <label x="116.84" y="160.02" size="1.778" layer="95"/>
 </segment>
-<segment>
-<pinref part="JP8" gate="G$1" pin="1"/>
-<wire x1="121.92" y1="12.7" x2="127" y2="12.7" width="0.1524" layer="91"/>
-<label x="127" y="12.7" size="1.778" layer="95"/>
-</segment>
 </net>

Commit message: working on embedded side code
Connections:
- net N$11 renamed VIN
Changed lines of the file:
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@@
 </segment>
 </net>
-<net name="N$11" class="0">
+<net name="VIN" class="0">
 <segment>
 <pinref part="U1" gate="VREG" pin="VIN"/>
