File: hardware/rev1/sw-4416-project-v1.sch (EAGLE design)
At the start: 56 parts, among them IC1 MCP73831, U1 ADP3338, X1 USB-MICROB, Y1 16M

Commit message: open sourcing hardware and software
Other:
- note added: "Attribution 3.0 Unported License. To view a copy of this"
- note added: "Copyright (c) 2013 Sean Watson"
- note added: "This work is licensed under the Creative Commons"
- note added: "license, visit http://creativecommons.org/licenses/by/3.0/"
Changed lines of the file:
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@@
 <text x="109.22" y="35.56" size="2.54" layer="94">Debug</text>
 <text x="172.72" y="2.54" size="2.54" layer="94" rot="MR0" align="center">Sep 24/12</text>
+<text x="134.62" y="53.34" size="1.778" layer="94">Copyright (c) 2013 Sean Watson</text>
+<text x="134.62" y="50.8" size="1.778" layer="94">This work is licensed under the Creative Commons</text>
+<text x="134.62" y="48.26" size="1.778" layer="94">Attribution 3.0 Unported License. To view a copy of this</text>
+<text x="134.62" y="45.72" size="1.778" layer="94">license, visit http://creativecommons.org/licenses/by/3.0/</text>
 </plain>
 <instances>
