File: hardware/rev2/sw-4416-project-v2.brd (EAGLE design)
At the start: 58.7 x 24.4 mm, 22 parts, among them U1 ADXL335, U2 MCP73831, X1 USB-MICROB, Y1 16M

Commit message: rev2 design done
Parts:
- added C10, C8, C9: 4.7u, SparkFun:0603-CAP
- added J1: CON_HEADER_PRG_AVR_ICSP", dp_devices:HEADER_PRG_2X03_SMD
- U$3: value 16M -> CRYSTAL_SMT
- moved R1 4.20 mm to (13.0, 15.2)
- moved R3 4.10 mm to (10.2, 19.3), turned to 180 degrees
- moved U2 4.06 mm to (10.2, 21.8)
- moved R2 3.39 mm to (13.0, 16.8), turned to 180 degrees
- moved U$2 3.31 mm to (42.2, 12.2)
- moved C4 2.30 mm to (29.5, 18.3), turned to 0 degrees
- moved S1 2.09 mm to (1.78, 7.11)
- moved X1 1.55 mm to (1.52, 16.8)
- moved C6 1.02 mm to (18.8, 2.54)
- moved R5 0.72 mm to (23.4, 5.84)
- moved JP1 0.57 mm to (9.65, 13.0)
- moved VREG1 0.51 mm to (9.65, 5.08)
- renumbered Y1 to U$3
Connections:
- removed net N$25: C1.2, C2.2, C3.2, C4.2, C5.2, C6.2, C7.2, JP1.2, R3.1, R4.1, U$1.15, U$1.23, U$1.35, U$1.43, U$1.5, U$2.1, U$2.12, U$2.25, U$2.27, U$2.28, U$2.29, U1.6, U2.2, VREG1.1, X1.GND
- new net GND: C1.2, C10.2, C2.2, C3.2, C4.2, C5.2, C6.2, C7.2, C8.2, C9.2, J1.6, JP1.2, R3.1, R4.1, U$1.15, U$1.23, U$1.35, U$1.43, U$1.5, U$2.1, U$2.12, U$2.25, U$2.27, U$2.28, U$2.29, U$3.2, U$3.4, U1.6, U2.2, VREG1.1, X1.GND
- net 3.3V: now also C10.1, C8.1, J1.2
- net MISO: now also J1.1
- net MOSI: now also J1.4
- net RST: now also J1.5
- net SCK: now also J1.3
- net VCC: now also C9.1
Routing:
- net GND: track 0.00 -> 204.9 mm, vias 0 -> 6
- net N$25: track 196.5 -> 0.00 mm, vias 8 -> 1
- net RST: track 0.00 -> 23.8 mm, vias 0 -> 1
- net MOSI: track 0.00 -> 16.3 mm, vias 0 -> 1
- net SCK: track 0.00 -> 14.4 mm, vias 0 -> 1
- net 3.3V: track 94.2 -> 108.4 mm
- net MISO: track 0.00 -> 11.4 mm, vias 0 -> 1
- net N$3: track 15.6 -> 8.56 mm
- net N$2: track 13.5 -> 8.50 mm
- net VCC: track 25.3 -> 29.5 mm
- net USB_D-: track 4.16 -> 6.72 mm
- net BT_TX: track 19.6 -> 17.2 mm
- net N$1: track 8.93 -> 6.64 mm
- net N$7: track 26.8 -> 25.3 mm
- net YOUT: track 12.1 -> 10.7 mm
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- added copper zone on layer 1, net GND
- added copper zone on layer 16, net GND
Other:
- board size 58.7 x 24.4 mm -> 58.7 x 25.1 mm

Commit message: second rev completed
Parts:
- added LED1: (no value), SparkFun:LED-0603
- added R6: 330, SparkFun:0603-RES
- VREG1: value (none) -> ADP3338
- flipped J1 to the bottom
Connections:
- new net N$27: LED1.C, R6.2
- net 3.3V: now also LED1.A
- net GND: now also R6.1
Routing:
- net RST: track 23.8 -> 13.1 mm
- net GND: track 204.9 -> 195.3 mm
- net 3.3V: track 108.4 -> 117.2 mm, vias 4 -> 5
- net MISO: track 11.4 -> 18.0 mm
- net N$27: track 0.00 -> 1.68 mm
- net SCK: track 14.4 -> 15.8 mm
- net MOSI: track 16.3 -> 16.9 mm

Commit message: open sourcing hardware and software
Other:
- board text added: "Copyright (c) 2013 Sean Watson"
- board text added: "This work is licensed under the Creative Commons Attribution 3.0 Unported License."
- board text added: "To view a copy of this license, visit http://creativecommons.org/licenses/by/3.0/."
Changed lines of the file:
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@@
 <layer number="23" name="tOrigins" color="15" fill="1" visible="yes" active="yes"/>
 <layer number="24" name="bOrigins" color="15" fill="1" visible="no" active="yes"/>
-<layer number="25" name="tNames" color="7" fill="1" visible="no" active="yes"/>
+<layer number="25" name="tNames" color="7" fill="1" visible="yes" active="yes"/>
 <layer number="26" name="bNames" color="7" fill="1" visible="no" active="yes"/>
 <layer number="27" name="tValues" color="7" fill="1" visible="yes" active="yes"/>
@@
 <hole x="52.324" y="2.794" drill="1.5"/>
 <hole x="4.318" y="23.114" drill="1.5"/>
+<text x="-0.254" y="-3.81" size="1.778" layer="25">Copyright (c) 2013 Sean Watson</text>
+<text x="-0.508" y="-8.89" size="1.778" layer="25">To view a copy of this license, visit http://creativecommons.org/licenses/by/3.0/.</text>
+<text x="-0.508" y="-6.35" size="1.778" layer="25">This work is licensed under the Creative Commons Attribution 3.0 Unported License.</text>
 </plain>
 <attributes>
