File: hardware/rev2/sw-4416-project-v2.sch (EAGLE design)
At the start: 22 parts, among them U1 ADXL335, U2 MCP73831, X1 USB-MICROB, Y1 16M

Commit message: rev2 design done
Parts:
- removed Y1: 16M, SparkFun:CRYSTAL5X3
- added C10, C8, C9: 4.7u, SparkFun:CAP0603-CAP
- added J1: CON_HEADER_PRG_AVR_ICSP", dp_devices:CON_HEADER_PRG_AVR_ICSP"
- added U$3: CRYSTAL_SMT, SparkFun:CRYSTAL_SMT
Connections:
- removed net N$25: C1.2, C2.2, C3.2, C4.2, C5.2, C6.2, C7.2, JP1.2, R3.1, R4.1, U$1.GND@15, U$1.GND@23, U$1.GND@35, U$1.GND@43, U$1.UGND, U$2.GND, U$2.GND1, U$2.GND2, U$2.GND3, U$2.GND4, U$2.GND5, U1.COM@6, U2.VSS, VREG1.GND, X1.GND
- new net GND: C1.2, C10.2, C2.2, C3.2, C4.2, C5.2, C6.2, C7.2, C8.2, C9.2, J1.GND, JP1.2, R3.1, R4.1, U$1.GND@15, U$1.GND@23, U$1.GND@35, U$1.GND@43, U$1.UGND, U$2.GND, U$2.GND1, U$2.GND2, U$2.GND3, U$2.GND4, U$2.GND5, U$3G$2.GND, U1.COM@6, U2.VSS, VREG1.GND, X1.GND
- net 3.3V: now also C10.1, C8.1, J1.+V
- net MISO: now also J1.MISO
- net MOSI: now also J1.MOSI
- net N$10: now also U$3G$1.1; no longer Y1.1
- net N$9: now also U$3G$1.2; no longer Y1.2
- net RST: now also J1.RST
- net SCK: now also J1.SCK
- net VCC: now also C9.1
Other:
- note added: "ICSP"
- moved on the sheet: JP1, R3, S1, U2

Commit message: second rev completed
Parts:
- added LED1: (no value), SparkFun:LED0603
- added R6: 330, SparkFun:RESISTOR0603-RES
- VREG1: value (none) -> ADP3338
Connections:
- new net N$27: LED1.C, R6.2
- net 3.3V: now also LED1.A
- net GND: now also R6.1
Other:
- note added: "LED"
Changed lines of the file:
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@@
 <setting verticaltext="up"/>
 </settings>
-<grid distance="0.1" unitdist="inch" unit="inch" style="lines" multiple="1" display="yes" altdistance="0.01" altunitdist="inch" altunit="inch"/>
+<grid distance="0.1" unitdist="inch" unit="inch" style="lines" multiple="1" display="no" altdistance="0.01" altunitdist="inch" altunit="inch"/>
 <layers>
 <layer number="1" name="Top" color="4" fill="1" visible="no" active="no"/>
@@
 <part name="X1" library="SparkFun" deviceset="USB" device="-MICROB"/>
 <part name="U$2" library="SparkFun" deviceset="BLUETOOTH-RN41" device="&quot;"/>
-<part name="VREG1" library="dp_devices" deviceset="VREG_3PINS" device="-SOT-223"/>
+<part name="VREG1" library="dp_devices" deviceset="VREG_3PINS" device="-SOT-223" value="ADP3338"/>
 <part name="U2" library="SparkFun" deviceset="MCP73831" device=""/>
 <part name="S1" library="SparkFun" deviceset="SWITCH-SPST" device="-SMD-A"/>
@@
 <part name="GND20" library="SparkFun" deviceset="GND" device=""/>
 <part name="U$3" library="SparkFun" deviceset="CRYSTAL_SMT" device=""/>
+<part name="P+9" library="SparkFun" deviceset="3.3V" device=""/>
+<part name="R6" library="SparkFun" deviceset="RESISTOR" device="0603-RES" value="330"/>
+<part name="GND21" library="SparkFun" deviceset="GND" device=""/>
+<part name="LED1" library="SparkFun" deviceset="LED" device="0603"/>
 </parts>
 <sheets>
@@
 <wire x1="177.8" y1="76.2" x2="177.8" y2="101.6" width="0.4064" layer="94"/>
 <text x="137.16" y="96.52" size="2.54" layer="94">ICSP</text>
+<wire x1="83.82" y1="83.82" x2="101.6" y2="83.82" width="0.4064" layer="94"/>
+<wire x1="101.6" y1="83.82" x2="101.6" y2="45.72" width="0.4064" layer="94"/>
+<wire x1="101.6" y1="45.72" x2="83.82" y2="45.72" width="0.4064" layer="94"/>
+<wire x1="83.82" y1="45.72" x2="83.82" y2="83.82" width="0.4064" layer="94"/>
+<text x="86.36" y="76.2" size="2.54" layer="94">LED</text>
 </plain>
 <instances>
@@
 <instance part="U$3" gate="G$1" x="15.24" y="111.76"/>
 <instance part="U$3" gate="G$2" x="15.24" y="96.52"/>
+<instance part="P+9" gate="G$1" x="93.98" y="76.2"/>
+<instance part="R6" gate="G$1" x="93.98" y="58.42" rot="R90"/>
+<instance part="GND21" gate="1" x="93.98" y="48.26"/>
+<instance part="LED1" gate="G$1" x="93.98" y="71.12"/>
 </instances>
 <busses>
@@
 <pinref part="P+8" gate="G$1" pin="3.3V"/>
 <wire x1="170.18" y1="93.98" x2="170.18" y2="91.44" width="0.1524" layer="91"/>
+</segment>
+<segment>
+<pinref part="P+9" gate="G$1" pin="3.3V"/>
+<pinref part="LED1" gate="G$1" pin="A"/>
+<wire x1="93.98" y1="76.2" x2="93.98" y2="73.66" width="0.1524" layer="91"/>
 </segment>
 </net>
@@
 <wire x1="22.86" y1="101.6" x2="22.86" y2="99.06" width="0.1524" layer="91"/>
 </segment>
+<segment>
+<pinref part="R6" gate="G$1" pin="1"/>
+<pinref part="GND21" gate="1" pin="GND"/>
+<wire x1="93.98" y1="53.34" x2="93.98" y2="50.8" width="0.1524" layer="91"/>
+</segment>
 </net>
 <net name="N$1" class="0">
@@
 </segment>
 </net>
+<net name="N$27" class="0">
+<segment>
+<pinref part="LED1" gate="G$1" pin="C"/>
+<pinref part="R6" gate="G$1" pin="2"/>
+<wire x1="93.98" y1="66.04" x2="93.98" y2="63.5" width="0.1524" layer="91"/>
+</segment>
+</net>

Commit message: open sourcing hardware and software
Other:
- note added: "Copyright (c) 2013 Sean Watson"
- note added: "This work is licensed under the Creative Commons Attribution 3.0 Unported License"
- note added: "To view a copy of this license, visit http://creativecommons.org/licenses/by/3.0/."
Changed lines of the file:
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@@
 <wire x1="83.82" y1="45.72" x2="83.82" y2="83.82" width="0.4064" layer="94"/>
 <text x="86.36" y="76.2" size="2.54" layer="94">LED</text>
+<text x="5.08" y="22.86" size="1.778" layer="94">Copyright (c) 2013 Sean Watson</text>
+<text x="5.08" y="20.32" size="1.778" layer="94">This work is licensed under the Creative Commons Attribution 3.0 Unported License</text>
+<text x="5.08" y="17.78" size="1.778" layer="94">To view a copy of this license, visit http://creativecommons.org/licenses/by/3.0/.</text>
 </plain>
 <instances>
